File: o3s7mobo/_autosave-o3s7mobo.kicad_pcb (KiCad board)
At the start: 4 copper layers, 330 x 217 mm, 45 parts, among them M1541 M1541, M1543 M1543

Commit message: Added Socket 7 schematics
I'm willing to have these schematics uploaded to the official KiCAD repositories; I'm just unsure how.
Connections:
- CPU1 pad A23: (no net) -> Net-(CPU1-PadA19)
- CPU1 pad A25: (no net) -> Net-(CPU1-PadA19)
- CPU1 pad A27: (no net) -> Net-(CPU1-PadA19)
- CPU1 pad A29: (no net) -> Net-(CPU1-PadA19)
- CPU1 pad AA37: (no net) -> Net-(CPU1-PadA19)
- CPU1 pad AC37: (no net) -> Net-(CPU1-PadA19)
- CPU1 pad AE37: (no net) -> Net-(CPU1-PadA19)
- CPU1 pad AG37: (no net) -> Net-(CPU1-PadA19)
- CPU1 pad AJ19: (no net) -> Net-(CPU1-PadA19)
- CPU1 pad AJ29: (no net) -> Net-(CPU1-PadA19)
- CPU1 pad AN21: (no net) -> Net-(CPU1-PadA19)
- CPU1 pad AN23: (no net) -> Net-(CPU1-PadA19)
- CPU1 pad AN25: (no net) -> Net-(CPU1-PadA19)
- CPU1 pad AN27: (no net) -> Net-(CPU1-PadA19)
- CPU1 pad AN29: (no net) -> Net-(CPU1-PadA19)
- CPU1 pad E21: (no net) -> Net-(CPU1-PadA19)
- CPU1 pad E27: (no net) -> Net-(CPU1-PadA19)
- CPU1 pad E37: (no net) -> Net-(CPU1-PadA19)
- CPU1 pad G37: (no net) -> Net-(CPU1-PadA19)
- CPU1 pad J37: (no net) -> Net-(CPU1-PadA19)
- CPU1 pad L33: (no net) -> Net-(CPU1-PadA19)
- CPU1 pad L37: (no net) -> Net-(CPU1-PadA19)
- CPU1 pad N37: (no net) -> Net-(CPU1-PadA19)
- CPU1 pad Q37: (no net) -> Net-(CPU1-PadA19)
- CPU1 pad S37: (no net) -> Net-(CPU1-PadA19)
- CPU1 pad T34: (no net) -> Net-(CPU1-PadA19)
- CPU1 pad U33: (no net) -> Net-(CPU1-PadA19)
- CPU1 pad U37: (no net) -> Net-(CPU1-PadA19)
- CPU1 pad W37: (no net) -> Net-(CPU1-PadA19)
- CPU1 pad Y37: (no net) -> Net-(CPU1-PadA19)
Routing:
- net GND: track 387.7 -> 547.4 mm
- net (no net): track 90.2 -> 0.00 mm
- net Net-(CPU1-PadA19): track 104.1 -> 115.7 mm
